Commit message: Rover: a machined vehicle instead of a box on four cylinders, visual only
The rover was a grey box with four black cylinders. It now has a chamfered
hull, a solar deck with structural ribs, bolt flanges and an inset array, a
sensor mast with a stereo camera head, an HGA dish, a whip antenna, radiators,
cable runs, an equipment box, and wheels with grousers, hub and rim - all
procedurally generated by mesh_gen/generate_rover_meshes.py (numpy + PIL only,
same dependency-free approach as the rock meshes), with committed OBJ assets
and procedural PBR atlases.

Every part is an additional <visual> on an EXISTING link. No new links, no new
joints, no mass: a massless link would be a dynamics risk, and every M3/M4
number in PROGRESS.md was measured against the current rover. Whole vehicle is
~4,340 triangles.

test_physics_untouched_in_sdf.py diffs the xacro-to-SDF output with <visual>
stripped against a baseline captured from the pristine pre-task tree -
independent ground truth rather than something derived from these edits. It
passes byte-identical on collisions, inertials, joints, sensors and plugin
parameters, and was watched go red on a deliberate mu1 change and again on a
chassis_mass change.

The find worth keeping, documented in the xacro: urdf2sdf silently emits
<diffuse>0 0 0 1</diffuse> for every visual after the FIRST on a multi-visual
link when the material is referenced by name only, regardless of which
material is named; an inline <color> on the reference works around it. Because
that tint multiplies the PBR albedo map, the deck, mast, dish, antenna,
equipment box, radiators and cable runs all rendered pure black while the hull
(first visual) and the wheels (sole visual on their links) were always
correct.

That cost real time, and the reason is worth recording: the symptom was read
as "a flat deck under a grazing sun is simply dim", which is physically
plausible and wrong. What settled it was proving that the intervention which
should have worked under that theory - near-white albedo plus aggressive
relief - produced a pixel-identical render. Also noted: urdf2sdf scales URDF
material colours by 1.25 and clamps at 1.0, so any channel above 0.8
saturates.

File: planetary/regolith_rover_description/urdf/regolith_rover.urdf.xacro (robot description, xacro)
@@ -9,4 +9,20 @@
        regolith_bringup's README for the gz service calls to start/stop it. -->
   <xacro:arg name="record_video" default="false"/>
+  <!-- Camera that exists only to film the rover, off by default ("none"). It is a
+       SEPARATE sensor from the onboard camera above on purpose: the perception suite
+       (RGB + depth on camera_link) is what the rover navigates with and its pose and
+       intrinsics are load-bearing, so footage requirements must never be met by moving
+       it. Two presets, both 1280x720 with the CameraVideoRecorder plugin on their own
+       service:
+         onboard - a mast looking forward over the deck, so the chassis and front
+                   wheels sit in the bottom of frame. Without that foreground there is
+                   no parallax and the footage reads as a still (see docs/media).
+         chase   - a boom behind and above, framing the whole rover in its terrain -
+                   for showing what the rover BODY does, e.g. bogging down and
+                   escaping.
+       Enable with cine_camera:=onboard|chase|both. 'both' films one run from both
+       angles at once - worth the extra render cost when what you want on film
+       (a rover bogging down) happens when it happens and cannot be re-staged. -->
+  <xacro:arg name="cine_camera" default="none"/>
   <!-- Leo-Rover-sized 4-wheel skid-steer chassis.
        Widened track + lowered chassis (vs. an earlier, narrower revision) after
@@ -22,6 +38,66 @@
   <xacro:property name="wheel_separation" value="0.46"/>
   <xacro:property name="wheelbase" value="0.28"/>
+  <!-- VISUAL ONLY below this point unless noted otherwise: procedurally generated by
+       regolith_rover_description/mesh_gen/generate_rover_meshes.py, committed under
+       meshes/. $(find ...) is resolved by xacro at process time (see hello_moon.launch's
+       _bake_rover_model_sdf: it runs `gz sdf -p` on the ALREADY-xacro-processed URDF, so
+       this becomes a literal file:// path baked into the SDF, not a runtime package://
+       lookup) to the installed share directory - meshes must be installed by
+       CMakeLists.txt (they are) and the workspace must be built + sourced before this
+       resolves, same as for any other change to this file.
+       Every part mounted on "chassis" shares ONE texture atlas (chassis_atlas_*.png) and
+       every wheel shares ONE texture atlas (wheel_atlas_*.png): verified with
+       `xacro regolith_rover.urdf.xacro | gz sdf -p -` that sdformat's urdf2sdf pass
+       applies a `<gazebo reference="LINK"><visual><material>` override to EVERY SDF
+       visual under that link regardless of the inner <visual name="...">  given - the
+       name is not used to pick a target - so a link with several decorative parts can
+       only ever be given one shared PBR material, never one per part. The different
+       "materials" you see per part (aluminum hull, gold MLI, solar cell, white
+       composite) are different UV regions of that one shared atlas, not different SDF
+       materials. -->
+  <xacro:property name="mesh_dir" value="file://$(find regolith_rover_description)/meshes"/>
   <material name="regolith_grey">
     <color rgba="0.55 0.55 0.58 1.0"/>
+  </material>
+  <!-- Named for what it now is: a mostly-white thermal deck plate with a small dark
+       cell array inset, not the dark solar panel it used to be.
+       IMPORTANT, verified with `xacro | gz sdf -p -`: on a link with several <visual>
+       elements (every decorative part here is on "chassis"), only the FIRST visual's
+       <material name="X"/> reference actually resolves X's <color> into the converted
+       SDF's <diffuse>/<ambient> - every later visual that references a material BY
+       NAME ONLY gets <diffuse>0 0 0 1</diffuse> instead (confirmed directly: built a
+       3-visual test case, visual 1 = name-only ref -> came out (0,0,0,1); visual 2 =
+       INLINE <color> on its own <material> tag -> came out correctly non-zero). Since
+       this diffuse/ambient value tints the PBR albedo_map rather than being ignored in
+       favour of it, every decorative visual past the first one on "chassis" was
+       rendering as a near-black silhouette REGARDLESS of its procedural texture or
+       geometry - this, not grazing sun angle or too-shallow relief, was the actual
+       cause of "the deck (and mast, dish, whip, equipment box, radiators, cable runs)
+       read as a black slab". Fix: every visual below now puts <color> INLINE on its
+       own <material> tag instead of only referencing one of these top-level
+       definitions by name. The top-level definitions stay (for the hull, which is the
+       first visual and needs no workaround, and as the canonical color values the
+       inline copies below are kept equal to).
+       One more converter quirk worth knowing when picking values here: urdf2sdf
+       scales each URDF color channel by 1.25 and clamps at 1.0 before writing
+       <diffuse>/<ambient> - confirmed against 4 independent channel values in the
+       converted SDF (0.55->0.6875, 0.12->0.15, 0.08->0.1, 0.85->1.0, all exactly
+       channel*1.25 up to the clamp). Practically: any channel above 0.8 saturates to
+       1.0 in Gazebo regardless of its exact URDF value - e.g. deck_white's 0.85/0.86/
+       0.88 all come out as flat 1.0 in the SDF, not as a slightly-off-white. Harmless
+       here since these are meant to read as bright anyway, but not the value you'd
+       compute by eye from the URDF color alone if the intent were a specific,
+       non-saturated tint. -->
+  <material name="deck_white">
+    <color rgba="0.85 0.86 0.88 1.0"/>
+  </material>
+  <material name="composite_white">
+    <color rgba="0.75 0.75 0.78 1.0"/>
+  </material>
+  <material name="harness_dark">
+    <color rgba="0.12 0.12 0.12 1.0"/>
+  </material>
+  <material name="mli_gold">
+    <color rgba="0.62 0.44 0.14 1.0"/>
   </material>
   <material name="wheel_black">
@@ -35,9 +111,100 @@
   </joint>
   <link name="chassis">
-    <visual>
-      <geometry>
-        <box size="${chassis_length} ${chassis_width} ${chassis_height}"/>
+    <!-- Machined hull: REPLACES the old flat box visual with the procedural mesh, same
+         origin, same footprint - the box <collision> right below is untouched. -->
+    <visual>
+      <geometry>
+        <mesh filename="${mesh_dir}/chassis_hull.obj"/>
       </geometry>
       <material name="regolith_grey"/>
+    </visual>
+    <!-- Everything below is EXTRA decoration: additional <visual> elements on the same
+         "chassis" link, each with its own <origin> offset and no <collision> of its
+         own - exactly the sanctioned mechanism for mast/dish/antenna/etc. per this
+         file's frozen-physics constraint. -->
+    <visual>
+      <!-- Raised on 4 visible corner standoffs (built into the mesh) above the hull
+           top (0.055) by DECK_STANDOFF_GAP (0.012) - see build_solar_deck's docstring:
+           an earlier ~1mm gap with hidden standoffs read as an unsupported floating
+           plate. -->
+      <origin xyz="0 0 0.067" rpy="0 0 0"/>
+      <geometry>
+        <mesh filename="${mesh_dir}/solar_deck.obj"/>
+      </geometry>
+      <material name="deck_white"><color rgba="0.85 0.86 0.88 1.0"/></material>
+    </visual>
+    <visual>
+      <!-- Sensor mast: base sits on the deck top (0.067 + 0.010 deck thickness =
+           0.077), mounted toward the rear so the camera head (built facing local +X)
+           looks forward over the chassis. Shortened from an earlier pass that added
+           ~0.44 m above the deck and visually dominated a 0.40 m vehicle - pole + yoke
+           + head + sunshade now add ~0.21 m, comfortably inside the "<= ~0.5 m above
+           the deck" budget and proportioned like a sensor head rather than a flagpole. -->
+      <origin xyz="-0.10 0 0.077" rpy="0 0 0"/>
+      <geometry>
+        <mesh filename="${mesh_dir}/mast_assembly.obj"/>
+      </geometry>
+      <material name="composite_white"><color rgba="0.75 0.75 0.78 1.0"/></material>
+    </visual>
+    <visual>
+      <!-- High-gain antenna dish, rear deck, tilted up and outboard. -->
+      <origin xyz="-0.15 0.10 0.086" rpy="0.0 -0.7 0.5"/>
+      <geometry>
+        <mesh filename="${mesh_dir}/dish.obj"/>
+      </geometry>
+      <material name="composite_white"><color rgba="0.75 0.75 0.78 1.0"/></material>
+    </visual>
+    <visual>
+      <!-- Whip antenna, rear corner. Short (0.13 m) and thick (1 cm base radius) on
+           purpose - see build_whip_antenna's docstring on why a needle-thin taper
+           disappears at shot scale. -->
+      <origin xyz="-0.18 -0.15 0.058" rpy="0.12 0.06 0"/>
+      <geometry>
+        <mesh filename="${mesh_dir}/whip_antenna.obj"/>
+      </geometry>
+      <material name="composite_white"><color rgba="0.75 0.75 0.78 1.0"/></material>
+    </visual>
+    <visual>
+      <!-- MLI-wrapped avionics box on the deck: a second, geometrically distinct gold
+           patch so the thermal-blanket material reads from angles where the hull skirt
+           is foreshortened or in shadow. -->
+      <origin xyz="-0.05 0.10 0.1015" rpy="0 0 0.35"/>
+      <geometry>
+        <mesh filename="${mesh_dir}/equipment_box.obj"/>
+      </geometry>
+      <material name="mli_gold"><color rgba="0.62 0.44 0.14 1.0"/></material>
+    </visual>
+    <visual>
+      <!-- Radiator panels, flush on the +Y/-Y side faces (see build_radiator's
+           docstring for why a pure yaw flip is enough to mount the same mesh on both
+           sides with no extra axis remap). -->
+      <origin xyz="0.05 ${chassis_width/2.0 + 0.003} -0.01" rpy="0 0 0"/>
+      <geometry>
+        <mesh filename="${mesh_dir}/radiator.obj"/>
+      </geometry>
+      <material name="composite_white"><color rgba="0.75 0.75 0.78 1.0"/></material>
+    </visual>
+    <visual>
+      <origin xyz="0.05 ${-chassis_width/2.0 - 0.003} -0.01" rpy="0 0 3.14159"/>
+      <geometry>
+        <mesh filename="${mesh_dir}/radiator.obj"/>
+      </geometry>
+      <material name="composite_white"><color rgba="0.75 0.75 0.78 1.0"/></material>
+    </visual>
+    <visual>
+      <!-- Cable harness run, front-right chamfer. -->
+      <origin xyz="0.10 0.14 0.045" rpy="0 0 1.9"/>
+      <geometry>
+        <mesh filename="${mesh_dir}/cable_run.obj"/>
+      </geometry>
+      <material name="harness_dark"><color rgba="0.12 0.12 0.12 1.0"/></material>
+    </visual>
+    <visual>
+      <!-- Cable harness run, front-left chamfer (mirrored). -->
+      <origin xyz="0.10 -0.14 0.045" rpy="0 0 -1.9"/>
+      <geometry>
+        <mesh filename="${mesh_dir}/cable_run.obj"/>
+      </geometry>
+      <material name="harness_dark"><color rgba="0.12 0.12 0.12 1.0"/></material>
     </visual>
     <collision>
@@ -58,12 +225,34 @@
     </inertial>
   </link>
+  <!-- One shared PBR material for every visual on "chassis" (see the mesh_dir property
+       comment above for why this has to be exactly one <gazebo reference> block: the
+       <visual name="..."> here is NOT used to target a specific chassis visual - it
+       gets applied to all of them - confirmed against actual `gz sdf -p` output. -->
+  <gazebo reference="chassis">
+    <visual name="chassis_atlas_material">
+      <material>
+        <pbr>
+          <metal>
+            <albedo_map>${mesh_dir}/chassis_atlas_albedo.png</albedo_map>
+            <normal_map>${mesh_dir}/chassis_atlas_normal.png</normal_map>
+            <roughness_map>${mesh_dir}/chassis_atlas_roughness.png</roughness_map>
+            <metalness_map>${mesh_dir}/chassis_atlas_metalness.png</metalness_map>
+          </metal>
+        </pbr>
+      </material>
+    </visual>
+  </gazebo>
   <xacro:macro name="wheel" params="prefix x_pos y_pos">
     <link name="${prefix}_wheel">
+      <!-- REPLACES the plain cylinder with the procedural grouser/rim/hub mesh, same
+           origin+rpy (the mesh is authored with its lathe axis along local Z, exactly
+           like the cylinder it replaces) - the cylinder <collision> right below is
+           untouched. -->
       <visual>
         <origin xyz="0 0 0" rpy="1.5708 0 0"/>
         <geometry>
-          <cylinder radius="${wheel_radius}" length="${wheel_width}"/>
+          <mesh filename="${mesh_dir}/wheel_hub.obj"/>
         </geometry>
-        <material name="wheel_black"/>
+        <material name="wheel_black"><color rgba="0.08 0.08 0.08 1.0"/></material>
       </visual>
       <collision>
@@ -94,4 +283,23 @@
       <mu1>1.4</mu1>
       <mu2>1.4</mu2>
+    </gazebo>
+    <!-- Separate <gazebo reference> block, purely so the friction block above (which
+         must not change - frozen physics) stays a clean untouched diff. One shared
+         wheel texture atlas, same reasoning as the chassis block above; here there is
+         only ever one visual per wheel link so the per-part-material limitation does
+         not bite, but the mechanism is the same. -->
+    <gazebo reference="${prefix}_wheel">
+      <visual name="${prefix}_wheel_atlas_material">
+        <material>
+          <pbr>
+            <metal>
+              <albedo_map>${mesh_dir}/wheel_atlas_albedo.png</albedo_map>
+              <normal_map>${mesh_dir}/wheel_atlas_normal.png</normal_map>
+              <roughness_map>${mesh_dir}/wheel_atlas_roughness.png</roughness_map>
+              <metalness_map>${mesh_dir}/wheel_atlas_metalness.png</metalness_map>
+            </metal>
+          </pbr>
+        </material>
+      </visual>
     </gazebo>
   </xacro:macro>
@@ -173,4 +381,50 @@
     </sensor>
   </gazebo>
+  <!-- See the cine_camera arg at the top of this file. Rigidly fixed to the chassis,
+       so the horizon pitches and rolls with the rover - that motion is the point. -->
+  <xacro:macro name="cine_cam" params="name xyz rpy hfov rate service">
+    <link name="${name}_link"/>
+    <joint name="${name}_joint" type="fixed">
+      <parent link="chassis"/>
+      <child link="${name}_link"/>
+      <origin xyz="${xyz}" rpy="${rpy}"/>
+    </joint>
+    <gazebo reference="${name}_link">
+      <sensor name="${name}" type="camera">
+        <always_on>true</always_on>
+        <update_rate>${rate}</update_rate>
+        <topic>${name}</topic>
+        <camera>
+          <horizontal_fov>${hfov}</horizontal_fov>
+          <image>
+            <width>1280</width>
+            <height>720</height>
+          </image>
+          <clip>
+            <near>0.05</near>
+            <far>200</far>
+          </clip>
+        </camera>
+        <plugin filename="gz-sim-camera-video-recorder-system" name="gz::sim::systems::CameraVideoRecorder">
+          <service>${service}</service>
+        </plugin>
+      </sensor>
+    </gazebo>
+  </xacro:macro>
+  <xacro:if value="${'$(arg cine_camera)' in ('onboard', 'both')}">
+    <xacro:cine_cam name="cine_camera" xyz="-0.25 0 0.42" rpy="0 0.38 0" hfov="1.4" rate="30"
+                    service="rover/cine/record_video"/>
+  </xacro:if>
+  <xacro:if value="${'$(arg cine_camera)' in ('chase', 'both')}">
+    <!-- Boom pose is set by what has to FIT, not by taste. At the original
+         (-1.6, 1.0, pitch 0.5, hfov 1.05) a 1.6 m boulder 1.3 m in front of the rover
+         had its top 7.6 deg ABOVE the frame's top edge: the footage showed only the
+         rock's dark underside next to its own cast shadow, and a rover stopped dead
+         against an obstacle nobody could see - it read as "immobilised on a shadow".
+         Pulled back and tilted up so the whole boulder is in shot (its top lands ~11%
+         down the frame, the rover ~70% down). -->
+    <xacro:cine_cam name="cine_chase" xyz="-2.6 0 1.1" rpy="0 0.24 0" hfov="1.3" rate="15"
+                    service="rover/chase/record_video"/>
+  </xacro:if>
   <gazebo>
     <allow_auto_disable>false</allow_auto_disable>
